Commit message: update support gripper

File: arctos_description/urdf/arctos.urdf (robot description, URDF)
Before this commit: robot arctos_description, 7 links, 6 joints
Links:
- removed link U_1
- removed link V_1
- removed link W_1
- removed link X_1
- removed link Y_1
- removed link Z_1
- added link Gripper_1, mass 0.5810486809925093; collision mesh filename=package://arctos_description/meshes/Gripper_1.stl scale=0.001 0.001 0.001; visual mesh filename=package://arctos_description/meshes/Gripper_1.stl scale=0.001 0.001 0.001
- added link Left_jaw_1, mass 0.07369602565859415; collision mesh filename=package://arctos_description/meshes/Left_jaw_1.stl scale=0.001 0.001 0.001; visual mesh filename=package://arctos_description/meshes/Left_jaw_1.stl scale=0.001 0.001 0.001
- added link Link_1_1, mass 10.394711633971145; collision mesh filename=package://arctos_description/meshes/Link_1_1.stl scale=0.001 0.001 0.001; visual mesh filename=package://arctos_description/meshes/Link_1_1.stl scale=0.001 0.001 0.001
- added link Link_2_1, mass 11.558090086674309; collision mesh filename=package://arctos_description/meshes/Link_2_1.stl scale=0.001 0.001 0.001; visual mesh filename=package://arctos_description/meshes/Link_2_1.stl scale=0.001 0.001 0.001
- added link Link_3_1, mass 3.601405589552794; collision mesh filename=package://arctos_description/meshes/Link_3_1.stl scale=0.001 0.001 0.001; visual mesh filename=package://arctos_description/meshes/Link_3_1.stl scale=0.001 0.001 0.001
- added link Link_4_1, mass 3.7852887653107565; collision mesh filename=package://arctos_description/meshes/Link_4_1.stl scale=0.001 0.001 0.001; visual mesh filename=package://arctos_description/meshes/Link_4_1.stl scale=0.001 0.001 0.001
- added link Link_5_1, mass 0.8319811655030993; collision mesh filename=package://arctos_description/meshes/Link_5_1.stl scale=0.001 0.001 0.001; visual mesh filename=package://arctos_description/meshes/Link_5_1.stl scale=0.001 0.001 0.001
- added link Link_6_1, mass 0.10343478090890781; collision mesh filename=package://arctos_description/meshes/Link_6_1.stl scale=0.001 0.001 0.001; visual mesh filename=package://arctos_description/meshes/Link_6_1.stl scale=0.001 0.001 0.001
- added link Right_jaw_1, mass 0.07312902168719511; collision mesh filename=package://arctos_description/meshes/Right_jaw_1.stl scale=0.001 0.001 0.001; visual mesh filename=package://arctos_description/meshes/Right_jaw_1.stl scale=0.001 0.001 0.001
- link base_link: mass 7.210677442504244 -> 7.598577592821282
Joints:
- removed joint Joint_1
- removed joint Joint_2
- removed joint Joint_3
- removed joint Joint_4
- removed joint Joint_5
- removed joint Joint_6
- added joint gripper: type fixed, parent Link_6_1, child Gripper_1, origin xyz=0.0 -0.006085 0.0 rpy=0 0 0
- added joint jaw1: type prismatic, parent Gripper_1, child Left_jaw_1, origin xyz=0.007741 -0.039998 0.029551 rpy=0 0 0, axis -0.0 0.0 -1.0, limit lower=0.0 upper=0.015 effort=100.0 velocity=100.0
- added joint jaw2: type prismatic, parent Gripper_1, child Right_jaw_1, origin xyz=0.007741 -0.039998 -0.030449 rpy=0 0 0, axis 0.0 -0.0 1.0, limit lower=0.0 upper=0.015 effort=100.0 velocity=100.0
- added joint joint1: type continuous, parent base_link, child Link_1_1, origin xyz=0.0 0.000529 0.111 rpy=0 0 0, axis -0.0 0.0 1.0
- added joint joint2: type continuous, parent Link_1_1, child Link_2_1, origin xyz=-0.05713 -0.020885 0.178378 rpy=0 0 0, axis 1.0 -0.0 -0.0
- added joint joint3: type continuous, parent Link_2_1, child Link_3_1, origin xyz=0.10013 0.001311 0.261007 rpy=0 0 0, axis -1.0 -0.0 0.0
- added joint joint4: type continuous, parent Link_3_1, child Link_4_1, origin xyz=-0.042999 -0.139695 0.021705 rpy=0 0 0, axis -0.0 1.0 -0.0
- added joint joint5: type continuous, parent Link_4_1, child Link_5_1, origin xyz=-0.039012 -0.121187 -0.001774 rpy=0 0 0, axis -1.0 -0.0 0.0
- added joint joint6: type continuous, parent Link_5_1, child Link_6_1, origin xyz=0.039204 -0.033835 0.0 rpy=0 0 0, axis -0.0 1.0 -0.0

File: arctos_description/urdf/materials.xacro (robot description, xacro)
@@ -1,6 +1,9 @@
 <?xml version="1.0" ?>
-<robot name="arctos_arm" xmlns:xacro="http://www.ros.org/wiki/xacro" >
-<material name="silver">
+<robot name="arctos_urdf" xmlns:xacro="http://www.ros.org/wiki/xacro" >
+<material name="silver_default">
   <color rgba="0.700 0.700 0.700 1.000"/>
 </material>
+<material name="paint_metallic_blue_2">
+  <color rgba="0.7764705882352941 0.7764705882352941 0.7764705882352941 1.0"/>
+</material>
 </robot>

Commit message: Included controller plugin

File: arctos_description/urdf/arctos.urdf (robot description, URDF)
Before this commit: robot arctos_urdf, 10 links, 9 joints
Joints:
- joint jaw1: limit lower=0.0 upper=0.015 effort=100.0 velocity=100.0 -> lower=0.0 upper=0.015 effort=100 velocity=100
- joint jaw2: limit lower=0.0 upper=0.015 effort=100.0 velocity=100.0 -> lower=0.0 upper=0.015 effort=100 velocity=100

File: arctos_description/urdf/arctos_urdf.xacro (robot description, xacro)
@@ -1,4 +1,4 @@
 <?xml version="1.0" ?>
-<robot name="arctos_urdf" xmlns:xacro="http://www.ros.org/wiki/xacro">
+<robot name="arctos" xmlns:xacro="http://www.ros.org/wiki/xacro">
 <xacro:include filename="$(find arctos_description)/urdf/materials.xacro" />
 <xacro:include filename="$(find arctos_description)/urdf/arctos_urdf.trans" />
@@ -259,3 +259,5 @@
   <limit upper="0.015" lower="0.0" effort="100" velocity="100"/>
 </joint>
+<xacro:include filename="$(find arctos_hardware_interface)/ros2_control/arctos.ros2_control.xacro" />
+<xacro:arctos_ros2_control name="arctos"/>
 </robot>

File: arctos_hardware_interface/ros2_control/arctos.ros2_control.xacro (robot description, xacro)
@@ -1,17 +1,101 @@
 <?xml version="1.0"?>
 <robot xmlns:xacro="http://www.ros.org/wiki/xacro">
-  <xacro:macro name="turck_encoder_driver" params="joint can_node_id can_topic_in can_topic_out vel_buf_size">
-    <ros2_control name="${joint}_encoder" type="sensor">
+  <xacro:macro name="arctos_ros2_control" params="name">
+    <ros2_control name="${name}" type="system">
       <hardware>
-        <plugin>turck_encoder_driver/EncoderInterface</plugin>
-        <param name="can_node_id">${can_node_id}</param>
-        <param name="can_topic_in">${can_topic_in}</param>
-        <param name="can_topic_out">${can_topic_out}</param>
-        <param name="vel_buf_size">${vel_buf_size}</param>
+        <plugin>arctos_interface/ArctosInterface</plugin>
       </hardware>
-      <joint name="${joint}">
-        <state_interface name="position"/>
+      <joint name="joint_1">
+        <command_interface name="position">
+          <param name="min">{-2*pi}</param>
+          <param name="max">{2*pi}</param>
+        </command_interface>
+        <command_interface name="velocity">
+          <param name="min">-3.15</param>
+          <param name="max">3.15</param>
+        </command_interface>
+        <state_interface name="position">
+          <param name="initial_value">0.0</param>
+        </state_interface>
         <state_interface name="velocity"/>
       </joint>
+      <joint name="joint_2">
+        <command_interface name="position">
+          <param name="min">{-2*pi}</param>
+          <param name="max">{2*pi}</param>
+        </command_interface>
+        <command_interface name="velocity">
+          <param name="min">-3.15</param>
+          <param name="max">3.15</param>
+        </command_interface>
+        <state_interface name="position">
+          <param name="initial_value">0.0</param>
+        </state_interface>
+        <state_interface name="velocity"/>
+      </joint>
+      <joint name="joint_3">
+        <command_interface name="position">
+          <param name="min">{-pi}</param>
+          <param name="max">{pi}</param>
+        </command_interface>
+        <command_interface name="velocity">
+          <param name="min">-3.15</param>
+          <param name="max">3.15</param>
+        </command_interface>
+        <state_interface name="position">
+          <param name="initial_value">0.0</param>
+        </state_interface>
+        <state_interface name="velocity"/>
+      </joint>
+      <joint name="joint_4">
+        <command_interface name="position">
+          <param name="min">{-2*pi}</param>
+          <param name="max">{2*pi}</param>
+        </command_interface>
+        <command_interface name="velocity">
+          <param name="min">-3.2</param>
+          <param name="max">3.2</param>
+        </command_interface>
+        <state_interface name="position">
+          <param name="initial_value">0.0</param>
+        </state_interface>
+        <state_interface name="velocity"/>
+      </joint>
+      <joint name="joint_5">
+        <command_interface name="position">
+          <param name="min">{-2*pi}</param>
+          <param name="max">{2*pi}</param>
+        </command_interface>
+        <command_interface name="velocity">
+          <param name="min">-3.2</param>
+          <param name="max">3.2</param>
+        </command_interface>
+        <state_interface name="position">
+          <param name="initial_value">0.0</param>
+        </state_interface>
+        <state_interface name="velocity"/>
+      </joint>
+      <joint name="joint_6">
+        <command_interface name="position">
+          <param name="min">{-2*pi}</param>
+          <param name="max">{2*pi}</param>
+        </command_interface>
+        <command_interface name="velocity">
+          <param name="min">-3.2</param>
+          <param name="max">3.2</param>
+        </command_interface>
+        <state_interface name="position">
+          <param name="initial_value">0.0</param>
+        </state_interface>
+        <state_interface name="velocity"/>
+      </joint>
+      <sensor name="tcp_fts_sensor">
+        <state_interface name="force.x"/>
+        <state_interface name="force.y"/>
+        <state_interface name="force.z"/>
+        <state_interface name="torque.x"/>
+        <state_interface name="torque.y"/>
+        <state_interface name="torque.z"/>
+      </sensor>
     </ros2_control>
   </xacro:macro>

File: arctos_moveit_config/config/arctos_urdf.ros2_control.xacro (robot description, xacro)
@@ -3,66 +3,63 @@
     <xacro:macro name="arctos_urdf_ros2_control" params="name initial_positions_file">
         <xacro:property name="initial_positions" value="${load_yaml(initial_positions_file)['initial_positions']}"/>
-        <ros2_control name="${name}" type="system">
-            <hardware>
-                <!-- By default, set up controllers for simulation. This won't work on real hardware -->
-                <plugin>mock_components/GenericSystem</plugin>
-            </hardware>
-            <joint name="joint1">
-                <command_interface name="position"/>
-                <state_interface name="position">
-                  <param name="initial_value">${initial_positions['joint1']}</param>
-                </state_interface>
-                <state_interface name="velocity"/>
-            </joint>
-            <joint name="joint2">
-                <command_interface name="position"/>
-                <state_interface name="position">
-                  <param name="initial_value">${initial_positions['joint2']}</param>
-                </state_interface>
-                <state_interface name="velocity"/>
-            </joint>
-            <joint name="joint3">
-                <command_interface name="position"/>
-                <state_interface name="position">
-                  <param name="initial_value">${initial_positions['joint3']}</param>
-                </state_interface>
-                <state_interface name="velocity"/>
-            </joint>
-            <joint name="joint4">
-                <command_interface name="position"/>
-                <state_interface name="position">
-                  <param name="initial_value">${initial_positions['joint4']}</param>
-                </state_interface>
-                <state_interface name="velocity"/>
-            </joint>
-            <joint name="joint5">
-                <command_interface name="position"/>
-                <state_interface name="position">
-                  <param name="initial_value">${initial_positions['joint5']}</param>
-                </state_interface>
-                <state_interface name="velocity"/>
-            </joint>
-            <joint name="joint6">
-                <command_interface name="position"/>
-                <state_interface name="position">
-                  <param name="initial_value">${initial_positions['joint6']}</param>
-                </state_interface>
-                <state_interface name="velocity"/>
-            </joint>
-            <joint name="jaw1">
-                <command_interface name="position"/>
-                <state_interface name="position">
-                  <param name="initial_value">${initial_positions['jaw1']}</param>
-                </state_interface>
-                <state_interface name="velocity"/>
-            </joint>
-            <joint name="jaw2">
-                <command_interface name="position"/>
-                <state_interface name="position">
-                  <param name="initial_value">${initial_positions['jaw2']}</param>
-                </state_interface>
-                <state_interface name="velocity"/>
-            </joint>
-        </ros2_control>
+        <ros2_control type="system">
+	    <hardware>
+	      <plugin>arctos_interface/ArctosInterface</plugin>
+	    </hardware>
+	    <joint name="joint1">
+	      <command_interface name="position"/>
+	      <state_interface name="position">
+		<param name="initial_value">0.0</param>
+	      </state_interface>
+	      <state_interface name="velocity">
+		<param name="initial_value">0.0</param>
+	      </state_interface>
+	    </joint>
+	    <joint name="joint2">
+	      <command_interface name="position"/>
+	      <state_interface name="position">
+		<param name="initial_value">0.0</param>
+	      </state_interface>
+	      <state_interface name="velocity">
+		<param name="initial_value">0.0</param>
+	      </state_interface>
+	    </joint>
+	    <joint name="joint3">
+	      <command_interface name="position"/>
+	      <state_interface name="position">
+		<param name="initial_value">0.0</param>
+	      </state_interface>
+	      <state_interface name="velocity">
+		<param name="initial_value">0.0</param>
+	      </state_interface>
+	    </joint>
+	    <joint name="joint4">
+	      <command_interface name="position"/>
+	      <state_interface name="position">
+		<param name="initial_value">0.0</param>
+	      </state_interface>
+	      <state_interface name="velocity">
+		<param name="initial_value">0.0</param>
+	      </state_interface>
+	    </joint>
+	    <joint name="joint5">
+	      <command_interface name="position"/>
+	      <state_interface name="position">
+		<param name="initial_value">0.0</param>
+	      </state_interface>
+	      <state_interface name="velocity">
+		<param name="initial_value">0.0</param>
+	      </state_interface>
+	    </joint>
+	    <joint name="joint6">
+	      <command_interface name="position"/>
+	      <state_interface name="position">
+		<param name="initial_value">0.0</param>
+	      </state_interface>
+	      <state_interface name="velocity">
+		<param name="initial_value">0.0</param>
+	      </state_interface>
+	    </joint>
+	</ros2_control>
     </xacro:macro>
 </robot>

Commit message: Small fix

File: arctos_description/urdf/arctos.urdf (robot description, URDF)
Before this commit: robot arctos_urdf, 10 links, 9 joints
Links:
- added link world
Joints:
- added joint base_joint: type fixed, parent world, child base_link, origin xyz=0 0 0 rpy=0 0 0, axis 0 0 1

File: arctos_description/urdf/arctos_urdf.xacro (robot description, xacro)
@@ -4,4 +4,11 @@
 <xacro:include filename="$(find arctos_description)/urdf/arctos_urdf.trans" />
 <xacro:include filename="$(find arctos_description)/urdf/arctos_urdf.gazebo" />
+<link name="world"/>
+<joint name="base_joint" type="fixed">
+    <parent link="world"/>
+    <child link="base_link"/>
+    <origin xyz="0 0 0" rpy="0 0 0"/>
+    <axis xyz="0 0 1"/>
+</joint>
 <link name="base_link">
   <inertial>

File: arctos_hardware_interface/ros2_control/arctos.ros2_control.xacro (robot description, xacro)
@@ -11,4 +11,8 @@
           <param name="max">{2*pi}</param>
         </command_interface>
+        <command_interface name="velocity">
+          <param name="min">-3.15</param>
+          <param name="max">3.15</param>
+        </command_interface>
         <state_interface name="position">
           <param name="initial_value">0.0</param>
@@ -20,4 +24,8 @@
           <param name="min">{-2*pi}</param>
           <param name="max">{2*pi}</param>
+        </command_interface>
+        <command_interface name="velocity">
+          <param name="min">-3.15</param>
+          <param name="max">3.15</param>
         </command_interface>
         <state_interface name="position">
@@ -31,4 +39,8 @@
           <param name="max">{pi}</param>
         </command_interface>
+        <command_interface name="velocity">
+          <param name="min">-3.15</param>
+          <param name="max">3.15</param>
+        </command_interface>
         <state_interface name="position">
           <param name="initial_value">0.0</param>
@@ -40,4 +52,8 @@
           <param name="min">{-2*pi}</param>
           <param name="max">{2*pi}</param>
+        </command_interface>
+        <command_interface name="velocity">
+          <param name="min">-3.2</param>
+          <param name="max">3.2</param>
         </command_interface>
         <state_interface name="position">
@@ -51,4 +67,8 @@
           <param name="max">{2*pi}</param>
         </command_interface>
+        <command_interface name="velocity">
+          <param name="min">-3.2</param>
+          <param name="max">3.2</param>
+        </command_interface>
         <state_interface name="position">
           <param name="initial_value">0.0</param>
@@ -60,4 +80,8 @@
           <param name="min">{-2*pi}</param>
           <param name="max">{2*pi}</param>
+        </command_interface>
+        <command_interface name="velocity">
+          <param name="min">-3.2</param>
+          <param name="max">3.2</param>
         </command_interface>
         <state_interface name="position">
