Commit message: Temp fix with launch files in description

File: arctos_description/urdf/arctos_urdf.xacro (robot description, xacro)
@@ -211,5 +211,5 @@
   </collision>
 </link>
-<joint name="joint1" type="continuous">
+<joint name="joint_1" type="continuous">
   <origin xyz="0.0 0.000529 0.111" rpy="0 0 0"/>
   <parent link="base_link"/>
@@ -217,5 +217,5 @@
   <axis xyz="-0.0 0.0 1.0"/>
 </joint>
-<joint name="joint2" type="continuous">
+<joint name="joint_2" type="continuous">
   <origin xyz="-0.05713 -0.020885 0.178378" rpy="0 0 0"/>
   <parent link="Link_1_1"/>
@@ -223,5 +223,5 @@
   <axis xyz="1.0 -0.0 -0.0"/>
 </joint>
-<joint name="joint3" type="continuous">
+<joint name="joint_3" type="continuous">
   <origin xyz="0.10013 0.001311 0.261007" rpy="0 0 0"/>
   <parent link="Link_2_1"/>
@@ -229,5 +229,5 @@
   <axis xyz="-1.0 -0.0 0.0"/>
 </joint>
-<joint name="joint4" type="continuous">
+<joint name="joint_4" type="continuous">
   <origin xyz="-0.042999 -0.139695 0.021705" rpy="0 0 0"/>
   <parent link="Link_3_1"/>
@@ -235,5 +235,5 @@
   <axis xyz="-0.0 1.0 -0.0"/>
 </joint>
-<joint name="joint5" type="continuous">
+<joint name="joint_5" type="continuous">
   <origin xyz="-0.039012 -0.121187 -0.001774" rpy="0 0 0"/>
   <parent link="Link_4_1"/>
@@ -246,5 +246,5 @@
   <child link="Gripper_1"/>
 </joint>
-<joint name="joint6" type="continuous">
+<joint name="joint_6" type="continuous">
   <origin xyz="0.039204 -0.033835 0.0" rpy="0 0 0"/>
   <parent link="Link_5_1"/>

File: arctos_hardware_interface/ros2_control/arctos.ros2_control.xacro (robot description, xacro)
@@ -16,5 +16,5 @@
         </command_interface>
         <state_interface name="position">
-          <param name="initial_value">0.0</param>
+          <param name="initial_value">0.0</param>arctos.ros2_control.xacro
         </state_interface>
         <state_interface name="velocity"/>
