Commit message: working controller

File: arctos_description/urdf/arctos.urdf.xacro (robot description, xacro)
@@ -1,455 +1,268 @@
 <?xml version="1.0" ?>
-<!-- =================================================================================== -->
-<!-- |    This document was autogenerated by xacro from arctos_urdf.xacro              | -->
-<!-- |    EDITING THIS FILE BY HAND IS NOT RECOMMENDED                                 | -->
-<!-- =================================================================================== -->
-<robot name="arctos">
-  <material name="silver_default">
-    <color rgba="0.700 0.700 0.700 1.000"/>
-  </material>
-  <material name="paint_metallic_blue_2">
-    <color rgba="0.7764705882352941 0.7764705882352941 0.7764705882352941 1.0"/>
-  </material>
-  <transmission name="joint_1_tran">
-    <type>transmission_interface/SimpleTransmission</type>
-    <joint name="joint_1">
-      <hardwareInterface>hardware_interface/EffortJointInterface</hardwareInterface>
-    </joint>
-    <actuator name="joint_1_actr">
-      <hardwareInterface>hardware_interface/EffortJointInterface</hardwareInterface>
-      <mechanicalReduction>1</mechanicalReduction>
-    </actuator>
-  </transmission>
-  <transmission name="joint_2_tran">
-    <type>transmission_interface/SimpleTransmission</type>
-    <joint name="joint_2">
-      <hardwareInterface>hardware_interface/EffortJointInterface</hardwareInterface>
-    </joint>
-    <actuator name="joint_2_actr">
-      <hardwareInterface>hardware_interface/EffortJointInterface</hardwareInterface>
-      <mechanicalReduction>1</mechanicalReduction>
-    </actuator>
-  </transmission>
-  <transmission name="joint_3_tran">
-    <type>transmission_interface/SimpleTransmission</type>
-    <joint name="joint_3">
-      <hardwareInterface>hardware_interface/EffortJointInterface</hardwareInterface>
-    </joint>
-    <actuator name="joint_3_actr">
-      <hardwareInterface>hardware_interface/EffortJointInterface</hardwareInterface>
-      <mechanicalReduction>1</mechanicalReduction>
-    </actuator>
-  </transmission>
-  <transmission name="joint_4_tran">
-    <type>transmission_interface/SimpleTransmission</type>
-    <joint name="joint_4">
-      <hardwareInterface>hardware_interface/EffortJointInterface</hardwareInterface>
-    </joint>
-    <actuator name="joint_4_actr">
-      <hardwareInterface>hardware_interface/EffortJointInterface</hardwareInterface>
-      <mechanicalReduction>1</mechanicalReduction>
-    </actuator>
-  </transmission>
-  <transmission name="joint_5_tran">
-    <type>transmission_interface/SimpleTransmission</type>
-    <joint name="joint_5">
-      <hardwareInterface>hardware_interface/EffortJointInterface</hardwareInterface>
-    </joint>
-    <actuator name="joint_5_actr">
-      <hardwareInterface>hardware_interface/EffortJointInterface</hardwareInterface>
-      <mechanicalReduction>1</mechanicalReduction>
-    </actuator>
-  </transmission>
-  <transmission name="joint_6_tran">
-    <type>transmission_interface/SimpleTransmission</type>
-    <joint name="joint_6">
-      <hardwareInterface>hardware_interface/EffortJointInterface</hardwareInterface>
-    </joint>
-    <actuator name="joint_6_actr">
-      <hardwareInterface>hardware_interface/EffortJointInterface</hardwareInterface>
-      <mechanicalReduction>1</mechanicalReduction>
-    </actuator>
-  </transmission>
-  <transmission name="jaw1_tran">
-    <type>transmission_interface/SimpleTransmission</type>
-    <joint name="jaw1">
-      <hardwareInterface>hardware_interface/EffortJointInterface</hardwareInterface>
-    </joint>
-    <actuator name="jaw1_actr">
-      <hardwareInterface>hardware_interface/EffortJointInterface</hardwareInterface>
-      <mechanicalReduction>1</mechanicalReduction>
-    </actuator>
-  </transmission>
-  <transmission name="jaw2_tran">
-    <type>transmission_interface/SimpleTransmission</type>
-    <joint name="jaw2">
-      <hardwareInterface>hardware_interface/EffortJointInterface</hardwareInterface>
-    </joint>
-    <actuator name="jaw2_actr">
-      <hardwareInterface>hardware_interface/EffortJointInterface</hardwareInterface>
-      <mechanicalReduction>1</mechanicalReduction>
-    </actuator>
-  </transmission>
-  <gazebo>
-    <plugin filename="libgazebo_ros_control.so" name="arctos_controller"/>
-  </gazebo>
-  <link name="world"/>
-  <joint name="base_joint" type="fixed">
+<robot name="arctos" xmlns:xacro="http://www.ros.org/wiki/xacro">
+<xacro:include filename="$(find arctos_description)/urdf/materials.xacro" />
+<xacro:include filename="$(find arctos_description)/urdf/arctos.ros2_control.xacro" />
+<xacro:arctos_ros2_control name="arctos"/>
+<link name="world"/>
+<joint name="base_joint" type="fixed">
     <parent link="world"/>
     <child link="base_link"/>
-    <origin rpy="0 0 0" xyz="0 0 0"/>
+    <origin xyz="0 0 0" rpy="0 0 0"/>
     <axis xyz="0 0 1"/>
-  </joint>
-  <link name="base_link">
-    <inertial>
-      <origin rpy="0 0 0" xyz="0.0009375030874740357 0.047087016508753216 0.06663230338123677"/>
-      <mass value="7.598577592821282"/>
-      <inertia ixx="0.063328" ixy="-0.000434" ixz="0.000108" iyy="0.03095" iyz="0.001366" izz="0.072371"/>
-    </inertial>
-    <visual>
-      <origin rpy="0 0 0" xyz="0 0 0"/>
-      <geometry>
-        <mesh filename="package://arctos_description/meshes/base_link.stl" scale="0.001 0.001 0.001"/>
-      </geometry>
-      <material name="paint_metallic_blue_2"/>
-    </visual>
-    <collision>
-      <origin rpy="0 0 0" xyz="0 0 0"/>
-      <geometry>
-        <mesh filename="package://arctos_description/meshes/base_link.stl" scale="0.001 0.001 0.001"/>
-      </geometry>
-    </collision>
-  </link>
-  <link name="Link_1_1">
-    <inertial>
-      <origin rpy="0 0 0" xyz="0.0022188890353287776 -0.004863444449475237 0.08546835509394825"/>
-      <mass value="10.394711633971145"/>
-      <inertia ixx="0.061139" ixy="0.00017" ixz="-0.00148" iyy="0.073854" iyz="0.003835" izz="0.05669"/>
-    </inertial>
-    <visual>
-      <origin rpy="0 0 0" xyz="-0.0 -0.000529 -0.111"/>
-      <geometry>
-        <mesh filename="package://arctos_description/meshes/Link_1_1.stl" scale="0.001 0.001 0.001"/>
-      </geometry>
-      <material name="paint_metallic_blue_2"/>
-    </visual>
-    <collision>
-      <origin rpy="0 0 0" xyz="-0.0 -0.000529 -0.111"/>
-      <geometry>
-        <mesh filename="package://arctos_description/meshes/Link_1_1.stl" scale="0.001 0.001 0.001"/>
-      </geometry>
-    </collision>
-  </link>
-  <link name="Link_2_1">
-    <inertial>
-      <origin rpy="0 0 0" xyz="0.055314283466519745 0.010843565259072822 0.11412354328486207"/>
-      <mass value="11.558090086674309"/>
-      <inertia ixx="0.128567" ixy="3e-06" ixz="0.001539" iyy="0.14463" iyz="-0.003293" izz="0.044463"/>
-    </inertial>
-    <visual>
-      <origin rpy="0 0 0" xyz="0.05713 0.020356 -0.289378"/>
-      <geometry>
-        <mesh filename="package://arctos_description/meshes/Link_2_1.stl" scale="0.001 0.001 0.001"/>
-      </geometry>
-      <material name="paint_metallic_blue_2"/>
-    </visual>
-    <collision>
-      <origin rpy="0 0 0" xyz="0.05713 0.020356 -0.289378"/>
-      <geometry>
-        <mesh filename="package://arctos_description/meshes/Link_2_1.stl" scale="0.001 0.001 0.001"/>
-      </geometry>
-    </collision>
-  </link>
-  <link name="Link_3_1">
-    <inertial>
-      <origin rpy="0 0 0" xyz="-0.04178369242643258 -0.03913025368943244 0.01221763827191602"/>
-      <mass value="3.601405589552794"/>
-      <inertia ixx="0.012497" ixy="-3.6e-05" ixz="-8.1e-05" iyy="0.006916" iyz="0.001536" izz="0.011789"/>
-    </inertial>
-    <visual>
-      <origin rpy="0 0 0" xyz="-0.043 0.019045 -0.550385"/>
-      <geometry>
-        <mesh filename="package://arctos_description/meshes/Link_3_1.stl" scale="0.001 0.001 0.001"/>
-      </geometry>
-      <material name="paint_metallic_blue_2"/>
-    </visual>
-    <collision>
-      <origin rpy="0 0 0" xyz="-0.043 0.019045 -0.550385"/>
-      <geometry>
-        <mesh filename="package://arctos_description/meshes/Link_3_1.stl" scale="0.001 0.001 0.001"/>
-      </geometry>
-    </collision>
-  </link>
-  <link name="Link_4_1">
-    <inertial>
-      <origin rpy="0 0 0" xyz="0.00021104999825562586 -0.06028834880207104 -0.0005408226217131773"/>
-      <mass value="3.7852887653107565"/>
-      <inertia ixx="0.011624" ixy="-9e-06" ixz="4e-06" iyy="0.011491" iyz="-7.1e-05" izz="0.017363"/>
-    </inertial>
-    <visual>
-      <origin rpy="0 0 0" xyz="-1e-06 0.15874 -0.57209"/>
-      <geometry>
-        <mesh filename="package://arctos_description/meshes/Link_4_1.stl" scale="0.001 0.001 0.001"/>
-      </geometry>
-      <material name="paint_metallic_blue_2"/>
-    </visual>
-    <collision>
-      <origin rpy="0 0 0" xyz="-1e-06 0.15874 -0.57209"/>
-      <geometry>
-        <mesh filename="package://arctos_description/meshes/Link_4_1.stl" scale="0.001 0.001 0.001"/>
-      </geometry>
-    </collision>
-  </link>
-  <link name="Link_5_1">
-    <inertial>
-      <origin rpy="0 0 0" xyz="0.0397291414278933 -0.012662394123331089 0.0007929187272999183"/>
-      <mass value="0.8319811655030993"/>
-      <inertia ixx="0.000732" ixy="-1.2e-05" ixz="5e-06" iyy="0.000958" iyz="-5e-06" izz="0.000907"/>
-    </inertial>
-    <visual>
-      <origin rpy="0 0 0" xyz="0.039011 0.279927 -0.570316"/>
-      <geometry>
-        <mesh filename="package://arctos_description/meshes/Link_5_1.stl" scale="0.001 0.001 0.001"/>
-      </geometry>
-      <material name="paint_metallic_blue_2"/>
-    </visual>
-    <collision>
-      <origin rpy="0 0 0" xyz="0.039011 0.279927 -0.570316"/>
-      <geometry>
-        <mesh filename="package://arctos_description/meshes/Link_5_1.stl" scale="0.001 0.001 0.001"/>
-      </geometry>
-    </collision>
-  </link>
-  <link name="Gripper_1">
-    <inertial>
-      <origin rpy="0 0 0" xyz="0.0036112727264542635 -0.014760653808445767 -0.00103677815369696"/>
-      <mass value="0.5810486809925093"/>
-      <inertia ixx="0.000385" ixy="1e-05" ixz="3e-06" iyy="0.000495" iyz="-2e-06" izz="0.000263"/>
-    </inertial>
-    <visual>
-      <origin rpy="0 0 0" xyz="-0.000193 0.319847 -0.570316"/>
-      <geometry>
-        <mesh filename="package://arctos_description/meshes/Gripper_1.stl" scale="0.001 0.001 0.001"/>
-      </geometry>
-      <material name="paint_metallic_blue_2"/>
-    </visual>
-    <collision>
-      <origin rpy="0 0 0" xyz="-0.000193 0.319847 -0.570316"/>
-      <geometry>
-        <mesh filename="package://arctos_description/meshes/Gripper_1.stl" scale="0.001 0.001 0.001"/>
-      </geometry>
-    </collision>
-  </link>
-  <link name="Link_6_1">
-    <inertial>
-      <origin rpy="0 0 0" xyz="6.567946382108388e-08 -0.003042398377876454 -3.032508957279134e-07"/>
-      <mass value="0.10343478090890781"/>
-      <inertia ixx="5.2e-05" ixy="-0.0" ixz="0.0" iyy="0.000103" iyz="0.0" izz="5.2e-05"/>
-    </inertial>
-    <visual>
-      <origin rpy="0 0 0" xyz="-0.000193 0.313762 -0.570316"/>
-      <geometry>
-        <mesh filename="package://arctos_description/meshes/Link_6_1.stl" scale="0.001 0.001 0.001"/>
-      </geometry>
-      <material name="paint_metallic_blue_2"/>
-    </visual>
-    <collision>
-      <origin rpy="0 0 0" xyz="-0.000193 0.313762 -0.570316"/>
-      <geometry>
-        <mesh filename="package://arctos_description/meshes/Link_6_1.stl" scale="0.001 0.001 0.001"/>
-      </geometry>
-    </collision>
-  </link>
-  <link name="Left_jaw_1">
-    <inertial>
-      <origin rpy="0 0 0" xyz="-0.011142702480351952 -0.009692440309284511 -0.009385792627785827"/>
-      <mass value="0.07369602565859415"/>
-      <inertia ixx="1.1e-05" ixy="2e-06" ixz="-0.0" iyy="6e-06" iyz="-0.0" izz="1.4e-05"/>
-    </inertial>
-    <visual>
-      <origin rpy="0 0 0" xyz="-0.007934 0.359845 -0.599867"/>
-      <geometry>
-        <mesh filename="package://arctos_description/meshes/Left_jaw_1.stl" scale="0.001 0.001 0.001"/>
-      </geometry>
-      <material name="paint_metallic_blue_2"/>
-    </visual>
-    <collision>
-      <origin rpy="0 0 0" xyz="-0.007934 0.359845 -0.599867"/>
-      <geometry>
-        <mesh filename="package://arctos_description/meshes/Left_jaw_1.stl" scale="0.001 0.001 0.001"/>
-      </geometry>
-    </collision>
-  </link>
-  <link name="Right_jaw_1">
-    <inertial>
-      <origin rpy="0 0 0" xyz="-0.008289104952972526 -0.009768535307719373 0.009395511902715814"/>
-      <mass value="0.07312902168719511"/>
-      <inertia ixx="1.1e-05" ixy="-1e-06" ixz="-1e-06" iyy="6e-06" iyz="0.0" izz="1.4e-05"/>
-    </inertial>
-    <visual>
-      <origin rpy="0 0 0" xyz="-0.007934 0.359845 -0.539867"/>
-      <geometry>
-        <mesh filename="package://arctos_description/meshes/Right_jaw_1.stl" scale="0.001 0.001 0.001"/>
-      </geometry>
-      <material name="paint_metallic_blue_2"/>
-    </visual>
-    <collision>
-      <origin rpy="0 0 0" xyz="-0.007934 0.359845 -0.539867"/>
-      <geometry>
-        <mesh filename="package://arctos_description/meshes/Right_jaw_1.stl" scale="0.001 0.001 0.001"/>
-      </geometry>
-    </collision>
-  </link>
-  <joint name="joint_1" type="continuous">
-    <origin rpy="0 0 0" xyz="0.0 0.000529 0.111"/>
-    <parent link="base_link"/>
-    <child link="Link_1_1"/>
-    <axis xyz="-0.0 0.0 1.0"/>
-  </joint>
-  <joint name="joint_2" type="continuous">
-    <origin rpy="0 0 0" xyz="-0.05713 -0.020885 0.178378"/>
-    <parent link="Link_1_1"/>
-    <child link="Link_2_1"/>
-    <axis xyz="1.0 -0.0 -0.0"/>
-  </joint>
-  <joint name="joint_3" type="continuous">
-    <origin rpy="0 0 0" xyz="0.10013 0.001311 0.261007"/>
-    <parent link="Link_2_1"/>
-    <child link="Link_3_1"/>
-    <axis xyz="-1.0 -0.0 0.0"/>
-  </joint>
-  <joint name="joint_4" type="continuous">
-    <origin rpy="0 0 0" xyz="-0.042999 -0.139695 0.021705"/>
-    <parent link="Link_3_1"/>
-    <child link="Link_4_1"/>
-    <axis xyz="-0.0 1.0 -0.0"/>
-  </joint>
-  <joint name="joint_5" type="continuous">
-    <origin rpy="0 0 0" xyz="-0.039012 -0.121187 -0.001774"/>
-    <parent link="Link_4_1"/>
-    <child link="Link_5_1"/>
-    <axis xyz="-1.0 -0.0 0.0"/>
-  </joint>
-  <joint name="gripper" type="fixed">
-    <origin rpy="0 0 0" xyz="0.0 -0.006085 0.0"/>
-    <parent link="Link_6_1"/>
-    <child link="Gripper_1"/>
-  </joint>
-  <joint name="joint_6" type="continuous">
-    <origin rpy="0 0 0" xyz="0.039204 -0.033835 0.0"/>
-    <parent link="Link_5_1"/>
-    <child link="Link_6_1"/>
-    <axis xyz="-0.0 1.0 -0.0"/>
-  </joint>
-  <joint name="jaw1" type="prismatic">
-    <origin rpy="0 0 0" xyz="0.007741 -0.039998 0.029551"/>
-    <parent link="Gripper_1"/>
-    <child link="Left_jaw_1"/>
-    <axis xyz="-0.0 0.0 -1.0"/>
-    <limit effort="100" lower="0.0" upper="0.015" velocity="100"/>
-  </joint>
-  <joint name="jaw2" type="prismatic">
-    <origin rpy="0 0 0" xyz="0.007741 -0.039998 -0.030449"/>
-    <parent link="Gripper_1"/>
-    <child link="Right_jaw_1"/>
-    <axis xyz="0.0 -0.0 1.0"/>
-    <limit effort="100" lower="0.0" upper="0.015" velocity="100"/>
-  </joint>
-  <ros2_control name="arctos" type="system">
-    <hardware>
-      <plugin>arctos_interface/ArctosInterface</plugin>
-    </hardware>
-    <joint name="joint_1">
-      <command_interface name="position">
-        <param name="min">{-2*pi}</param>
-        <param name="max">{2*pi}</param>
-      </command_interface>
-      <command_interface name="velocity">
-        <param name="min">-3.15</param>
-        <param name="max">3.15</param>
-      </command_interface>
-      <state_interface name="position">
-        <param name="initial_value">0.0</param>
-      </state_interface>
-      <state_interface name="velocity"/>
-    </joint>
-    <joint name="joint_2">
-      <command_interface name="position">
-        <param name="min">{-2*pi}</param>
-        <param name="max">{2*pi}</param>
-      </command_interface>
-      <command_interface name="velocity">
-        <param name="min">-3.15</param>
-        <param name="max">3.15</param>
-      </command_interface>
-      <state_interface name="position">
-        <param name="initial_value">0.0</param>
-      </state_interface>
-      <state_interface name="velocity"/>
-    </joint>
-    <joint name="joint_3">
-      <command_interface name="position">
-        <param name="min">{-pi}</param>
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