Commit message: update motor driver

File: arctos_description/urdf/materials.xacro (robot description, xacro)
@@ -1,9 +1,9 @@
-<?xml version="1.0" ?>
-<robot name="arctos_urdf" xmlns:xacro="http://www.ros.org/wiki/xacro" >
-<material name="silver_default">
-  <color rgba="0.700 0.700 0.700 1.000"/>
-</material>
-<material name="paint_metallic_blue_2">
-  <color rgba="0.7764705882352941 0.7764705882352941 0.7764705882352941 1.0"/>
-</material>
+<?xml version="1.0"?>
+<robot name="arctos" xmlns:xacro="http://www.ros.org/wiki/xacro">
+  <material name="white">
+    <color rgba="1.0 1.0 1.0 1.000" />
+  </material>
+  <material name="black">
+    <color rgba="0.0 0.0 0.0 1.0" />
+  </material>
 </robot>

File: arctos_hardware_interface/ros2_control/arctos.ros2_control.xacro (robot description, xacro)
@@ -4,7 +4,7 @@
     <ros2_control name="${name}" type="system">
       <hardware>
-        <plugin>arctos_interface/ArctosInterface</plugin>
+        <plugin>libarctos_interface.so</plugin>
       </hardware>
-      <joint name="joint_1">
+      <joint name="X_joint">
         <command_interface name="position">
           <param name="min">{-2*pi}</param>
@@ -20,5 +20,5 @@
         <state_interface name="velocity"/>
       </joint>
-      <joint name="joint_2">
+      <joint name="Y_joint">
         <command_interface name="position">
           <param name="min">{-2*pi}</param>
@@ -34,5 +34,5 @@
         <state_interface name="velocity"/>
       </joint>
-      <joint name="joint_3">
+      <joint name="Z_joint">
         <command_interface name="position">
           <param name="min">{-pi}</param>
@@ -48,5 +48,5 @@
         <state_interface name="velocity"/>
       </joint>
-      <joint name="joint_4">
+      <joint name="A_joint">
         <command_interface name="position">
           <param name="min">{-2*pi}</param>
@@ -62,5 +62,5 @@
         <state_interface name="velocity"/>
       </joint>
-      <joint name="joint_5">
+      <joint name="B_joint">
         <command_interface name="position">
           <param name="min">{-2*pi}</param>
@@ -76,5 +76,5 @@
         <state_interface name="velocity"/>
       </joint>
-      <joint name="joint_6">
+      <joint name="C_joint">
         <command_interface name="position">
           <param name="min">{-2*pi}</param>
